File: KiCad/BUS_CAN.kicad_sch (KiCad schematic)
At the start: 0 parts

Commit message: Esquematic BUS creat + Diagrama blocs v.3.
Parts:
- added C2: 100n, symbol Device:C
- added J1: DE9_Pins_MountingHoles, symbol Connector:DE9_Pins_MountingHoles
- added R3: 10k, symbol Device:R
- added R4: 120, symbol Device:R
- added U3: SN65HVD230, Package_SO:SOIC-8_3.9x4.9mm_P1.27mm, symbol Interface_CAN_LIN:SN65HVD230
Connections:
- new net: R3.2, U3.8 (Rs)
- new net CANH: J1.7, R4.2, U3.7 (CANH)
- new net CANL: J1.2, R4.1, U3.6 (CANL)
- new net CANRX: U3.4 (R)
- new net CANTX: U3.1 (D)
- new net GND_PWR: C2.2, J1.6, R3.1, U3.2 (GND)
- new net VDD_3V3: C2.1, U3.3 (VCC)
- no-connect marks 0 -> 8
Other:
- note added: "Pin Rs --> Resistencia 10k per slope control. Slew rate = 15V/us"

Commit message: aclaracions BUS CAN
Connections:
- no-connect marks 8 -> 6
Other:
- note added: "Falta USART"
- note added: "Pin Vref --> Output de Vcc/2"
Changed lines of the file:
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@@
 	(generator_version "9.0")
 	(paper "A4")
+	(text "Pin Vref --> Output de Vcc/2"
+		(exclude_from_sim no)
+		(at 84.328 64.516 0)
+		(effects
+			(font
+				(size 1.27 1.27)
+			)
+		)
+	)
 	(text "Pin Rs --> Resistencia 10k per slope control.\nSlew rate = 15V/us"
 		(exclude_from_sim no)
 		(at 96.52 78.486 0)
+		(effects
+			(font
+				(size 1.27 1.27)
+			)
+		)
+	)
+	(text "Falta USART\n"
+		(exclude_from_sim no)
+		(at 147.32 53.34 0)
 		(effects
 			(font
@@
 	)
 	(no_connect
-		(at 154.94 52.07)
-	)
-	(no_connect
-		(at 154.94 54.61)
-	)
-	(no_connect
