File: KiCad/INPUTS.kicad_sch (KiCad schematic)
At the start: 0 parts

Commit message: Actualització Sheet Inputs
Parts:
- added R5, R6, R7, R8: 10K, symbol Device:R
- added SW_UP, SW_UP1, SW_UP2, SW_UP3: SW_Push, symbol Switch:SW_Push
Connections:
- new net GND: SW_UP.2, SW_UP1.2, SW_UP2.2, SW_UP3.2
- new net MCLR: R8.2, SW_UP3.1
- new net VDD_3V3: R5.1, R6.1, R7.1, R8.1
- new net WIN_BTN_DOWN: R6.2, SW_UP1.1
- new net WIN_BTN_UP: R5.2, SW_UP.1
- new net WIN_LIMIT: R7.2, SW_UP2.1

Commit message: H
Parts:
- renumbered SW_UP to SW_UP4
Changed lines of the file:
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@@
 		(dnp no)
 		(fields_autoplaced yes)
-		(property "Reference" "SW_UP"
+		(property "Reference" "SW_UP4"
 			(at 186.69 55.88 0)
 			(effects
@@
 			(project "PROJECTE_EINES"
 				(path "/347831db-5db9-4aff-ad32-e56fd770e219/85b10b44-f8b7-4b58-879f-bd15e6c8e976"
-					(reference "SW_UP")
+					(reference "SW_UP4")
 					(unit 1)
 				)
