File: KiCad/INPUTS.kicad_sch (KiCad schematic)
At the start: 10 parts, among them SW1 SW_DPDT_x2, SW2 SW_DPDT_x2, SW4 SW_DPDT_x2

Commit message: V2 placement
Parts:
- removed R_LIMIT1: 10K, Resistor_SMD:R_0805_2012Metric, symbol Device:R
- removed SW1: SW_DPDT_x2, symbol Switch:SW_DPDT_x2
- removed unit 2 of SW2
- removed SW_UP2: SW_LIMIT, Button_Switch_SMD:SW_SPST_TL3342, symbol Switch:SW_Push
- SW2, SW4: footprint (none) -> Button_Switch_SMD:SW_DPDT_CK_JS202011JCQN
Connections:
- no-connect marks 6 -> 0

Commit message: V1 Routing
Parts:
- SW2: renamed from SW4; footprint Button_Switch_SMD:SW_DPDT_CK_JS202011JCQN -> Button_Switch_THT:SW_CK_JS202011CQN_DPDT_Straight
- renumbered SW2 to SW1
Changed lines of the file:
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@@
 	(polyline
 		(pts
-			(xy 130.81 12.065) (xy 130.81 64.77)
+			(xy 130.81 -8.255) (xy 130.81 64.77)
 		)
 		(stroke
@@
 		(dnp no)
 		(fields_autoplaced yes)
-		(property "Reference" "#PWR022"
+		(property "Reference" "#PWR023"
 			(at 105.41 41.91 0)
 			(effects
@@
 			(project "PROJECTE_EINES"
 				(path "/347831db-5db9-4aff-ad32-e56fd770e219/85b10b44-f8b7-4b58-879f-bd15e6c8e976"
-					(reference "#PWR022")
+					(reference "#PWR023")
 					(unit 1)
 				)
@@
 		(dnp no)
 		(fields_autoplaced yes)
-		(property "Reference" "#PWR023"
+		(property "Reference" "#PWR024"
 			(at 105.41 54.61 0)
 			(effects
@@
 			(project "PROJECTE_EINES"
 				(path "/347831db-5db9-4aff-ad32-e56fd770e219/85b10b44-f8b7-4b58-879f-bd15e6c8e976"
-					(reference "#PWR023")
+					(reference "#PWR024")
 					(unit 1)
 				)
@@
 		(dnp no)
 		(fields_autoplaced yes)
-		(property "Reference" "#PWR020"
+		(property "Reference" "#PWR022"
 			(at 76.2 52.07 0)
 			(effects
@@
 			(project "PROJECTE_EINES"
 				(path "/347831db-5db9-4aff-ad32-e56fd770e219/85b10b44-f8b7-4b58-879f-bd15e6c8e976"
-					(reference "#PWR020")
+					(reference "#PWR022")
 					(unit 1)
 				)
@@
 		(dnp no)
 		(fields_autoplaced yes)
-		(property "Reference" "#PWR019"
+		(property "Reference" "#PWR021"
 			(at 54.61 50.8 0)
 			(effects
@@
 			(project "PROJECTE_EINES"
 				(path "/347831db-5db9-4aff-ad32-e56fd770e219/85b10b44-f8b7-4b58-879f-bd15e6c8e976"
-					(reference "#PWR019")
+					(reference "#PWR021")
 					(unit 1)
 				)
@@
 		(dnp no)
 		(fields_autoplaced yes)
-		(property "Reference" "SW2"
+		(property "Reference" "SW1"
 			(at 87.63 36.83 0)
 			(effects
@@
 			(project "PROJECTE_EINES"
 				(path "/347831db-5db9-4aff-ad32-e56fd770e219/85b10b44-f8b7-4b58-879f-bd15e6c8e976"
-					(reference "SW2")
+					(reference "SW1")
 					(unit 1)
 				)
@@
 		(dnp no)
 		(fields_autoplaced yes)
-		(property "Reference" "#PWR018"
+		(property "Reference" "#PWR020"
 			(at 22.86 48.26 0)
 			(effects
@@
 			(project "PROJECTE_EINES"
 				(path "/347831db-5db9-4aff-ad32-e56fd770e219/85b10b44-f8b7-4b58-879f-bd15e6c8e976"
-					(reference "#PWR018")
+					(reference "#PWR020")
 					(unit 1)
 				)
@@
 		(dnp no)
 		(fields_autoplaced yes)
-		(property "Reference" "SW4"
+		(property "Reference" "SW2"
 			(at 179.07 31.75 0)
 			(effects
@@
 			)
 		)
-		(property "Footprint" "Button_Switch_SMD:SW_DPDT_CK_JS202011JCQN"
+		(property "Footprint" "Button_Switch_THT:SW_CK_JS202011CQN_DPDT_Straight"
 			(at 179.07 40.64 0)
 			(effects
@@
 			(project "PROJECTE_EINES"
 				(path "/347831db-5db9-4aff-ad32-e56fd770e219/85b10b44-f8b7-4b58-879f-bd15e6c8e976"
-					(reference "SW4")
-					(unit 1)
-				)
+					(reference "SW2")
+					(unit 1)
+				)

Commit message: Versió Final projecte
Parts:
- SW_UP1: value SW_MCLR -> SW
- renumbered R_MCLR1 to R4, R_BTNUP1 to R5, R_BTNDOWN1 to R6, R_Lock/Unlock1 to R7
Changed lines of the file:
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@@
 		(on_board yes)
 		(dnp no)
-		(property "Reference" "R_BTNUP1"
+		(property "Reference" "R5"
 			(at 95.758 33.02 0)
 			(effects
@@
 			(project "PROJECTE_EINES"
 				(path "/347831db-5db9-4aff-ad32-e56fd770e219/85b10b44-f8b7-4b58-879f-bd15e6c8e976"
-					(reference "R_BTNUP1")
+					(reference "R5")
 					(unit 1)
 				)
@@
 		(on_board yes)
 		(dnp no)
-		(property "Reference" "R_Lock/Unlock1"
+		(property "Reference" "R7"
 			(at 165.354 35.306 90)
 			(effects
@@
 			(project "PROJECTE_EINES"
 				(path "/347831db-5db9-4aff-ad32-e56fd770e219/85b10b44-f8b7-4b58-879f-bd15e6c8e976"
-					(reference "R_Lock/Unlock1")
+					(reference "R7")
 					(unit 1)
 				)
@@
 		(on_board yes)
 		(dnp no)
-		(property "Reference" "R_BTNDOWN1"
+		(property "Reference" "R6"
 			(at 100.584 46.482 0)
 			(effects
@@
 			(project "PROJECTE_EINES"
 				(path "/347831db-5db9-4aff-ad32-e56fd770e219/85b10b44-f8b7-4b58-879f-bd15e6c8e976"
-					(reference "R_BTNDOWN1")
+					(reference "R6")
 					(unit 1)
 				)
@@
 		(dnp no)
 		(fields_autoplaced yes)
-		(property "Reference" "R_MCLR1"
+		(property "Reference" "R4"
 			(at 34.29 38.1 90)
 			(effects
@@
 			(project "PROJECTE_EINES"
 				(path "/347831db-5db9-4aff-ad32-e56fd770e219/85b10b44-f8b7-4b58-879f-bd15e6c8e976"
-					(reference "R_MCLR1")
+					(reference "R4")
 					(unit 1)
 				)
@@
 			)
 		)
-		(property "Value" "SW_MCLR"
+		(property "Value" "SW"
 			(at 46.99 39.37 0)
 			(effects
