File: KiCad/SENSOR_RFID.kicad_sch (KiCad schematic)
At the start: 2 parts, among them J2 Conn_01x08_Pin

Commit message: Correció etapa d'alimentació e Inputs
Parts:
- renumbered C3 to C9, J2 to J3
Changed lines of the file:
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@@
 		(on_board yes)
 		(dnp no)
-		(property "Reference" "C3"
+		(property "Reference" "C9"
 			(at 157.48 80.01 90)
 			(effects
@@
 			(project ""
 				(path "/347831db-5db9-4aff-ad32-e56fd770e219/31dcd71e-4130-43cb-a335-13c9e1a3d043"
-					(reference "C3")
+					(reference "C9")
 					(unit 1)
 				)
@@
 		(dnp no)
 		(fields_autoplaced yes)
-		(property "Reference" "#PWR036"
+		(property "Reference" "#PWR021"
 			(at 166.37 82.55 0)
 			(effects
@@
 			(project ""
 				(path "/347831db-5db9-4aff-ad32-e56fd770e219/31dcd71e-4130-43cb-a335-13c9e1a3d043"
-					(reference "#PWR036")
+					(reference "#PWR021")
 					(unit 1)
 				)
@@
 		(dnp no)
 		(fields_autoplaced yes)
-		(property "Reference" "J2"
+		(property "Reference" "J3"
 			(at 147.955 53.34 0)
 			(effects
@@
 			(project ""
 				(path "/347831db-5db9-4aff-ad32-e56fd770e219/31dcd71e-4130-43cb-a335-13c9e1a3d043"
-					(reference "J2")
+					(reference "J3")
 					(unit 1)
 				)
@@
 		(dnp no)
 		(fields_autoplaced yes)
-		(property "Reference" "#PWR035"
+		(property "Reference" "#PWR020"
 			(at 166.37 74.93 0)
 			(effects
@@
 			(project ""
 				(path "/347831db-5db9-4aff-ad32-e56fd770e219/31dcd71e-4130-43cb-a335-13c9e1a3d043"
-					(reference "#PWR035")
-					(unit 1)
-				)
+					(reference "#PWR020")
+					(unit 1)
+				)

Commit message: Versió final Esquematic
Parts:
- C9: footprint Capacitor_SMD:C_0805_2012Metric_Pad1.18x1.45mm_HandSolder -> Capacitor_SMD:C_0805_2012Metric
Changed lines of the file:
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@@
 			)
 		)
-		(property "Footprint" "Capacitor_SMD:C_0805_2012Metric_Pad1.18x1.45mm_HandSolder"
+		(property "Footprint" "Capacitor_SMD:C_0805_2012Metric"
 			(at 161.29 75.2348 0)
 			(effects
