File: KiCad/MOTOR_FINESTRA.kicad_sch (KiCad schematic)
At the start: 7 parts, among them U3 VNH5019A-E

Commit message: Correció etapa d'alimentació e Inputs
Parts:
- renumbered C9 to C10, C10 to C11, R12 to R10, R1 to R8, R11 to R9, U3 to U5
Other:
- moved on the sheet: C12
Changed lines of the file:
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@@
+	(wire
+		(pts
+			(xy 154.94 81.28) (xy 142.24 81.28)
+		)
+		(stroke
+			(width 0)
+			(type default)
+		)
+	)
 	(wire
 		(pts
@@
 	(wire
 		(pts
-			(xy 157.48 82.55) (xy 158.75 82.55)
-		)
-		(stroke
-			(width 0)
-			(type default)
-		)
-	)
-	(wire
-		(pts
 			(xy 129.54 62.23) (xy 129.54 69.85)
 		)
@@
 		(pts
 			(xy 143.51 120.65) (xy 143.51 119.38)
-		)
-		(stroke
-			(width 0)
-			(type default)
-		)
-	)
-	(wire
-		(pts
-			(xy 157.48 81.28) (xy 142.24 81.28)
-		)
-		(stroke
-			(width 0)
-			(type default)
-		)
-	)
-	(wire
-		(pts
-			(xy 157.48 82.55) (xy 157.48 81.28)
 		)
 		(stroke
@@
 		(dnp no)
 		(fields_autoplaced yes)
-		(property "Reference" "#PWR037"
+		(property "Reference" "#PWR031"
 			(at 130.81 115.57 0)
 			(effects
@@
 			(project ""
 				(path "/347831db-5db9-4aff-ad32-e56fd770e219/b6effc59-48f1-49a7-95ce-6407716902cc"
-					(reference "#PWR037")
+					(reference "#PWR031")
 					(unit 1)
 				)
@@
 		(on_board yes)
 		(dnp no)
-		(property "Reference" "R12"
+		(property "Reference" "R10"
 			(at 181.864 89.408 90)
 			(effects
@@
 			(project "PROJECTE_EINES"
 				(path "/347831db-5db9-4aff-ad32-e56fd770e219/b6effc59-48f1-49a7-95ce-6407716902cc"
-					(reference "R12")
+					(reference "R10")
 					(unit 1)
 				)
@@
 		(on_board yes)
 		(dnp no)
-		(property "Reference" "#PWR039"
+		(property "Reference" "#PWR036"
 			(at 184.15 85.09 0)
 			(effects
@@
 			(project "PROJECTE_EINES"
 				(path "/347831db-5db9-4aff-ad32-e56fd770e219/b6effc59-48f1-49a7-95ce-6407716902cc"
-					(reference "#PWR039")
+					(reference "#PWR036")
 					(unit 1)
 				)
@@
 	(symbol
 		(lib_id "Device:C")
-		(at 162.56 82.55 270)
+		(at 158.75 81.28 270)
 		(unit 1)
 		(exclude_from_sim no)
@@
 		(fields_autoplaced yes)
 		(property "Reference" "C12"
-			(at 162.56 74.93 90)
+			(at 158.75 73.66 90)
 			(effects
 				(font
@@
 		)
 		(property "Value" "100nF"
-			(at 162.56 77.47 90)
+			(at 158.75 76.2 90)
 			(effects
 				(font
@@
 		)
 		(property "Footprint" ""
-			(at 158.75 83.5152 0)
+			(at 154.94 82.2452 0)
 			(effects
 				(font
@@
 		)
 		(property "Datasheet" "~"
-			(at 162.56 82.55 0)
+			(at 158.75 81.28 0)
 			(effects
 				(font
@@
 		)
 		(property "Description" "Unpolarized capacitor"
-			(at 162.56 82.55 0)
+			(at 158.75 81.28 0)
 			(effects
 				(font
@@
 		(dnp no)
 		(fields_autoplaced yes)
-		(property "Reference" "C10"
+		(property "Reference" "C11"
 			(at 133.35 62.23 90)
 			(effects
@@
 			(project "PROJECTE_EINES"
 				(path "/347831db-5db9-4aff-ad32-e56fd770e219/b6effc59-48f1-49a7-95ce-6407716902cc"
-					(reference "C10")
+					(reference "C11")
 					(unit 1)
 				)
@@
 		(on_board yes)
 		(dnp no)
-		(property "Reference" "R11"
+		(property "Reference" "R9"
 			(at 159.766 101.092 90)
 			(effects
@@
 			(project "PROJECTE_EINES"
 				(path "/347831db-5db9-4aff-ad32-e56fd770e219/b6effc59-48f1-49a7-95ce-6407716902cc"
-					(reference "R11")
+					(reference "R9")
 					(unit 1)
 				)
@@
 		(dnp no)
 		(fields_autoplaced yes)
-		(property "Reference" "#PWR01"
+		(property "Reference" "#PWR032"
 			(at 143.51 66.04 0)
 			(effects
@@
 			(project ""
 				(path "/347831db-5db9-4aff-ad32-e56fd770e219/b6effc59-48f1-49a7-95ce-6407716902cc"
-					(reference "#PWR01")
+					(reference "#PWR032")
 					(unit 1)
 				)
@@
 		(on_board yes)
 		(dnp no)
-		(property "Reference" "#PWR038"
+		(property "Reference" "#PWR034"
 			(at 157.48 99.06 0)
 			(effects
@@
 			(project ""
 				(path "/347831db-5db9-4aff-ad32-e56fd770e219/b6effc59-48f1-49a7-95ce-6407716902cc"
-					(reference "#PWR038")
+					(reference "#PWR034")
 					(unit 1)
 				)
@@
 		(dnp no)
 		(fields_autoplaced yes)
-		(property "Reference" "#PWR08"
+		(property "Reference" "#PWR033"
 			(at 143.51 125.73 0)
 			(effects
@@
 			(project "PROJECTE_EINES"
 				(path "/347831db-5db9-4aff-ad32-e56fd770e219/b6effc59-48f1-49a7-95ce-6407716902cc"
-					(reference "#PWR08")
+					(reference "#PWR033")
 					(unit 1)
 				)
@@
 		(dnp no)
 		(fields_autoplaced yes)
-		(property "Reference" "C9"
+		(property "Reference" "C10"
 			(at 133.35 54.61 90)
 			(effects
@@
 			(project ""
 				(path "/347831db-5db9-4aff-ad32-e56fd770e219/b6effc59-48f1-49a7-95ce-6407716902cc"
-					(reference "C9")
+					(reference "C10")
 					(unit 1)
 				)
@@
 		(dnp no)
 		(fields_autoplaced yes)
-		(property "Reference" "U3"
+		(property "Reference" "U5"
 			(at 134.2233 73.66 0)
 			(effects
@@
 			(project ""
 				(path "/347831db-5db9-4aff-ad32-e56fd770e219/b6effc59-48f1-49a7-95ce-6407716902cc"
-					(reference "U3")
+					(reference "U5")
 					(unit 1)
 				)
@@
 		(dnp no)
 		(fields_autoplaced yes)
-		(property "Reference" "R1"
+		(property "Reference" "R8"
 			(at 146.05 115.5699 0)
 			(effects
@@
 			(project ""
 				(path "/347831db-5db9-4aff-ad32-e56fd770e219/b6effc59-48f1-49a7-95ce-6407716902cc"
-					(reference "R1")
+					(reference "R8")
 					(unit 1)
 				)
@@
 	(symbol
 		(lib_id "power:GND")
-		(at 166.37 82.55 90)
+		(at 162.56 81.28 90)
 		(unit 1)
 		(exclude_from_sim no)
@@
 		(dnp no)
 		(fields_autoplaced yes)
-		(property "Reference" "#PWR04"
-			(at 172.72 82.55 0)
+		(property "Reference" "#PWR035"
+			(at 168.91 81.28 0)
 			(effects
 				(font
@@
 		)
 		(property "Value" "GND"
-			(at 170.18 82.5499 90)
+			(at 166.37 81.2799 90)
 			(effects
 				(font
@@
 		)
 		(property "Footprint" ""
-			(at 166.37 82.55 0)
+			(at 162.56 81.28 0)
 			(effects
 				(font
@@
 		)
 		(property "Datasheet" ""
-			(at 166.37 82.55 0)
+			(at 162.56 81.28 0)
 			(effects
 				(font
@@
 		)
 		(property "Description" "Power symbol creates a global label with name \"GND\" , ground"
-			(at 166.37 82.55 0)
+			(at 162.56 81.28 0)
 			(effects
 				(font
@@
 			(project "PROJECTE_EINES"
 				(path "/347831db-5db9-4aff-ad32-e56fd770e219/b6effc59-48f1-49a7-95ce-6407716902cc"
-					(reference "#PWR04")
+					(reference "#PWR035")
 					(unit 1)
 				)
@@
 		(dnp no)
 		(fields_autoplaced yes)
-		(property "Reference" "#PWR03"
+		(property "Reference" "#PWR030"
 			(at 115.57 96.52 0)
 			(effects
@@
 			(project "PROJECTE_EINES"
 				(path "/347831db-5db9-4aff-ad32-e56fd770e219/b6effc59-48f1-49a7-95ce-6407716902cc"
-					(reference "#PWR03")
-					(unit 1)
-				)
+					(reference "#PWR030")
+					(unit 1)
+				)

Commit message: Actualizació Footprints
Parts:
- C_WIN_1: renamed from C10; footprint (none) -> Capacitor_SMD:C_0805_2012Metric
- C_WIN_2: renamed from C11; footprint (none) -> Capacitor_SMD:C_1206_3216Metric
- C_WIN_CP1: renamed from C12; footprint (none) -> Capacitor_SMD:C_0805_2012Metric
- renumbered R8 to R_WIN_CS1, R10 to R_WIN_DIAGA1, R9 to R_WIN_DIAGB1
Other:
- moved on the sheet: R_WIN_DIAGA1, R_WIN_DIAGB1
