File: KiCad/ETAPA_POTENCIA.kicad_sch (KiCad schematic)
At the start: 15 parts, among them U1 LM2596S-5, U2 LM1117DT-3.3

Commit message: Versió final Esquematic
Parts:
- removed CIN1, COUT2, C_INBUCK1, C_OUTBUCK1: 100nF, Capacitor_SMD:C_0805_2012Metric, symbol Device:C
- removed CIN2, COUT1: 10uF, Capacitor_SMD:C_1206_3216Metric, symbol Device:C
- removed C_INBUCK2, C_OUTBUCK2: 220uF, Capacitor_SMD:CP_Elec_8x10, symbol Device:C
- removed D_OUTBUCK1, D_PROT1: D_Schottky, Diode_SMD:D_SMB_Modified, symbol Device:D_Schottky
- removed D_TVS1: D_TVS, Diode_SMD:D_SMB_Modified, symbol Device:D_TVS
- removed F_PROT1: Fuse, Fuse:Fuse_1812_4532Metric, symbol Device:Fuse
- removed L2: 33uH, Inductor_SMD:L_10.4x10.4_H4.8, symbol Device:L
- removed U1: LM2596S-5, Package_TO_SOT_SMD:TO-263-5_TabPin3, symbol Regulator_Switching:LM2596S-5
- removed U2: LM1117DT-3.3, Package_TO_SOT_SMD:TO-252-3_TabPin2, symbol Regulator_Linear:LM1117DT-3.3
