File: KiCad/ETAPA_ALIMENTACIO_sch.kicad_sch (KiCad schematic)
At the start: 14 parts

Commit message: Errors solucionats
Parts:
- gave numbers to parts that had none: 14
Connections:
- net VBAT_12V renamed +12V
