File: KiCad/ETAPA_ALIMENTACIO_sch.kicad_sch (KiCad schematic)
At the start: 14 parts

Commit message: V3 layout
Parts:
- gave numbers to parts that had none: 14
Changed lines of the file:
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@@
 		(dnp no)
 		(fields_autoplaced yes)
-		(property "Reference" "U?"
+		(property "Reference" "U4"
 			(at 185.42 76.2 0)
 			(effects
@@
 			(project "PROJECTE_EINES"
 				(path "/347831db-5db9-4aff-ad32-e56fd770e219/b8d025f8-884e-44af-b29b-4fb2140b95b4"
-					(reference "U?")
+					(reference "U4")
 					(unit 1)
 				)
@@
 		(dnp no)
 		(fields_autoplaced yes)
-		(property "Reference" "COUT?"
+		(property "Reference" "COUT1"
 			(at 200.66 87.6299 0)
 			(effects
@@
 			(project "PROJECTE_EINES"
 				(path "/347831db-5db9-4aff-ad32-e56fd770e219/b8d025f8-884e-44af-b29b-4fb2140b95b4"
-					(reference "COUT?")
+					(reference "COUT1")
 					(unit 1)
 				)
@@
 		(on_board yes)
 		(dnp no)
-		(property "Reference" "C_INBUCK?"
+		(property "Reference" "C_INBUCK2"
 			(at 102.87 75.438 0)
 			(effects
@@
 			(project "PROJECTE_EINES"
 				(path "/347831db-5db9-4aff-ad32-e56fd770e219/b8d025f8-884e-44af-b29b-4fb2140b95b4"
-					(reference "C_INBUCK?")
+					(reference "C_INBUCK2")
 					(unit 1)
 				)
@@
 		(dnp no)
 		(fields_autoplaced yes)
-		(property "Reference" "F_PROT?"
+		(property "Reference" "F_PROT1"
 			(at 66.04 71.12 90)
 			(effects
@@
 			(project "PROJECTE_EINES"
 				(path "/347831db-5db9-4aff-ad32-e56fd770e219/b8d025f8-884e-44af-b29b-4fb2140b95b4"
-					(reference "F_PROT?")
+					(reference "F_PROT1")
 					(unit 1)
 				)
@@
 		(dnp no)
 		(fields_autoplaced yes)
-		(property "Reference" "CIN?"
+		(property "Reference" "CIN1"
 			(at 177.8 87.6299 0)
 			(effects
@@
 			(project "PROJECTE_EINES"
 				(path "/347831db-5db9-4aff-ad32-e56fd770e219/b8d025f8-884e-44af-b29b-4fb2140b95b4"
-					(reference "CIN?")
+					(reference "CIN1")
 					(unit 1)
 				)
@@
 		(on_board yes)
 		(dnp no)
-		(property "Reference" "C_OUTBUCK?"
+		(property "Reference" "C_OUTBUCK2"
 			(at 160.528 91.948 0)
 			(effects
@@
 			(project "PROJECTE_EINES"
 				(path "/347831db-5db9-4aff-ad32-e56fd770e219/b8d025f8-884e-44af-b29b-4fb2140b95b4"
-					(reference "C_OUTBUCK?")
+					(reference "C_OUTBUCK2")
 					(unit 1)
 				)
@@
 		(dnp no)
 		(fields_autoplaced yes)
-		(property "Reference" "D_PROT?"
+		(property "Reference" "D_PROT1"
 			(at 77.7875 71.12 0)
 			(effects
@@
 			(project "PROJECTE_EINES"
 				(path "/347831db-5db9-4aff-ad32-e56fd770e219/b8d025f8-884e-44af-b29b-4fb2140b95b4"
-					(reference "D_PROT?")
+					(reference "D_PROT1")
 					(unit 1)
 				)
@@
 		(dnp no)
 		(fields_autoplaced yes)
-		(property "Reference" "L?"
+		(property "Reference" "L1"
 			(at 146.05 77.47 90)
 			(effects
@@
 			(project "PROJECTE_EINES"
 				(path "/347831db-5db9-4aff-ad32-e56fd770e219/b8d025f8-884e-44af-b29b-4fb2140b95b4"
-					(reference "L?")
+					(reference "L1")
 					(unit 1)
 				)
@@
 		(on_board yes)
 		(dnp no)
-		(property "Reference" "C_INBUCK?"
+		(property "Reference" "C_INBUCK1"
 			(at 90.932 75.438 0)
 			(effects
@@
 			(project "PROJECTE_EINES"
 				(path "/347831db-5db9-4aff-ad32-e56fd770e219/b8d025f8-884e-44af-b29b-4fb2140b95b4"
-					(reference "C_INBUCK?")
+					(reference "C_INBUCK1")
 					(unit 1)
 				)
@@
 		(dnp no)
 		(fields_autoplaced yes)
-		(property "Reference" "COUT?"
+		(property "Reference" "COUT2"
 			(at 212.09 87.6299 0)
 			(effects
@@
 			(project "PROJECTE_EINES"
 				(path "/347831db-5db9-4aff-ad32-e56fd770e219/b8d025f8-884e-44af-b29b-4fb2140b95b4"
-					(reference "COUT?")
+					(reference "COUT2")
 					(unit 1)
 				)
@@
 		(dnp no)
 		(fields_autoplaced yes)
-		(property "Reference" "#PWR?"
+		(property "Reference" "#PWR0102"
 			(at 214.63 86.36 0)
 			(effects
@@
 			(project "PROJECTE_EINES"
 				(path "/347831db-5db9-4aff-ad32-e56fd770e219/b8d025f8-884e-44af-b29b-4fb2140b95b4"
-					(reference "#PWR?")
+					(reference "#PWR0102")
 					(unit 1)
 				)
@@
 		(dnp no)
 		(fields_autoplaced yes)
-		(property "Reference" "D_TVS?"
+		(property "Reference" "D_TVS1"
 			(at 87.63 81.2799 90)
 			(effects
@@
 			(project "PROJECTE_EINES"
 				(path "/347831db-5db9-4aff-ad32-e56fd770e219/b8d025f8-884e-44af-b29b-4fb2140b95b4"
-					(reference "D_TVS?")
+					(reference "D_TVS1")
 					(unit 1)
 				)
@@
 		(on_board yes)
 		(dnp no)
-		(property "Reference" "C_OUTBUCK?"
+		(property "Reference" "C_OUTBUCK1"
 			(at 147.574 92.202 0)
 			(effects
@@
 			(project "PROJECTE_EINES"
 				(path "/347831db-5db9-4aff-ad32-e56fd770e219/b8d025f8-884e-44af-b29b-4fb2140b95b4"
-					(reference "C_OUTBUCK?")
+					(reference "C_OUTBUCK1")
 					(unit 1)
 				)
@@
 		(dnp no)
 		(fields_autoplaced yes)
-		(property "Reference" "U?"
+		(property "Reference" "U3"
 			(at 123.19 69.85 0)
 			(effects
@@
 			(project "PROJECTE_EINES"
 				(path "/347831db-5db9-4aff-ad32-e56fd770e219/b8d025f8-884e-44af-b29b-4fb2140b95b4"
-					(reference "U?")
+					(reference "U3")
 					(unit 1)
 				)
@@
 		(dnp no)
 		(fields_autoplaced yes)
-		(property "Reference" "#PWR?"
+		(property "Reference" "#PWR0101"
 			(at 180.34 104.14 0)
 			(effects
@@
 			(project "PROJECTE_EINES"
 				(path "/347831db-5db9-4aff-ad32-e56fd770e219/b8d025f8-884e-44af-b29b-4fb2140b95b4"
-					(reference "#PWR?")
+					(reference "#PWR0101")
 					(unit 1)
 				)
@@
 		(on_board yes)
 		(dnp no)
-		(property "Reference" "D_OUTBUCK?"
+		(property "Reference" "D_OUTBUCK1"
 			(at 135.382 92.456 90)
 			(effects
@@
 			(project "PROJECTE_EINES"
 				(path "/347831db-5db9-4aff-ad32-e56fd770e219/b8d025f8-884e-44af-b29b-4fb2140b95b4"
-					(reference "D_OUTBUCK?")
+					(reference "D_OUTBUCK1")
 					(unit 1)
 				)
@@
 		(dnp no)
 		(fields_autoplaced yes)
-		(property "Reference" "#PWR?"
+		(property "Reference" "#PWR0103"
 			(at 157.48 81.28 0)
 			(effects
@@
 			(project "PROJECTE_EINES"
 				(path "/347831db-5db9-4aff-ad32-e56fd770e219/b8d025f8-884e-44af-b29b-4fb2140b95b4"
-					(reference "#PWR?")
-					(unit 1)
-				)
+					(reference "#PWR0103")
+					(unit 1)
+				)
