File: KiCad/ETAPA_POTENICA.kicad_sch (KiCad schematic)
At the start: 14 parts, among them U3 VNH5019A-E, U5 VNH5019A-E

Commit message: Versio final KiCad, BOM i Diagrama de Blocs
Parts:
- removed R_CS_DOOR1: 1k, Resistor_SMD:R_0805_2012Metric, symbol Device:R
Connections:
- net +3.3V: now also U5.6 (CS_DIS)
- net GNDPWR: no longer U5.6 (CS_DIS)
- no-connect marks 0 -> 1
Other:
- note added: "Desactivació sensor de corrent"
- note added: "Sortida bomba de càrrega"
- note added: "Sortida sensor de corrent"
- note added: "Terminal CS desactivat"
- moved on the sheet: C_CP_DOOR1, C_VDD_DOOR1, C_VDD_DOOR2, C_WIN_1, C_WIN_2, C_WIN_CP1, R_DIAGA_DOOR1, R_DIAGB_DOOR1, R_WIN_CS1, R_WIN_DIAGA1, R_WIN_DIAGB1, U3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

Commit message: Versio final
Parts:
- C_VDD_DOOR2, C_WIN_2: footprint Capacitor_SMD:C_1206_3216Metric -> Capacitor_SMD:C_0805_2012Metric
Changed lines of the file:
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@@
 			)
 		)
-		(property "Footprint" "Capacitor_SMD:C_1206_3216Metric"
+		(property "Footprint" "Capacitor_SMD:C_0805_2012Metric"
 			(at 158.75 56.1848 0)
 			(effects
@@
 			)
 		)
-		(property "Footprint" "Capacitor_SMD:C_1206_3216Metric"
+		(property "Footprint" "Capacitor_SMD:C_0805_2012Metric"
 			(at 45.72 52.3748 0)
 			(effects

Commit message: Versió Final projecte
Parts:
- C15: renamed from C_VDD_DOOR2; footprint Capacitor_SMD:C_0805_2012Metric -> Capacitor_SMD:C_1206_3216Metric
- C9: renamed from C_WIN_2; footprint Capacitor_SMD:C_0805_2012Metric -> Capacitor_SMD:C_1206_3216Metric
- renumbered C_WIN_CP1 to C10, C_VDD_DOOR1 to C14, C_CP_DOOR1 to C18, C_WIN_1 to C8, R_WIN_DIAGA1 to R10, R_DIAGB_DOOR1 to R11, R_DIAGA_DOOR1 to R12, R_WIN_CS1 to R8, R_WIN_DIAGB1 to R9
Changed lines of the file:
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@@
 		(on_board yes)
 		(dnp no)
-		(property "Reference" "R_DIAGA_DOOR1"
+		(property "Reference" "R12"
 			(at 204.47 75.438 90)
 			(effects
@@
 			(project "PROJECTE_EINES"
 				(path "/347831db-5db9-4aff-ad32-e56fd770e219/0182dfdd-06e0-4cd2-9407-e3ad60659aa3"
-					(reference "R_DIAGA_DOOR1")
+					(reference "R12")
 					(unit 1)
 				)
@@
 		(on_board yes)
 		(dnp no)
-		(property "Reference" "#FLG03"
+		(property "Reference" "#FLG04"
 			(at 36.195 55.88 0)
 			(effects
@@
 			(project "PROJECTE_EINES"
 				(path "/347831db-5db9-4aff-ad32-e56fd770e219/0182dfdd-06e0-4cd2-9407-e3ad60659aa3"
-					(reference "#FLG03")
+					(reference "#FLG04")
 					(unit 1)
 				)
@@
 		(dnp no)
 		(fields_autoplaced yes)
-		(property "Reference" "C_WIN_CP1"
+		(property "Reference" "C10"
 			(at 60.96 57.15 90)
 			(effects
@@
 			(project "PROJECTE_EINES"
 				(path "/347831db-5db9-4aff-ad32-e56fd770e219/0182dfdd-06e0-4cd2-9407-e3ad60659aa3"
-					(reference "C_WIN_CP1")
+					(reference "C10")
 					(unit 1)
 				)
@@
 		(on_board yes)
 		(dnp no)
-		(property "Reference" "R_WIN_DIAGB1"
+		(property "Reference" "R9"
 			(at 94.996 84.074 90)
 			(effects
@@
 			(project "PROJECTE_EINES"
 				(path "/347831db-5db9-4aff-ad32-e56fd770e219/0182dfdd-06e0-4cd2-9407-e3ad60659aa3"
-					(reference "R_WIN_DIAGB1")
+					(reference "R9")
 					(unit 1)
 				)
@@
 		(on_board yes)
 		(dnp no)
-		(property "Reference" "C_VDD_DOOR1"
+		(property "Reference" "C14"
 			(at 161.544 43.942 90)
 			(effects
@@
 			(project "PROJECTE_EINES"
 				(path "/347831db-5db9-4aff-ad32-e56fd770e219/0182dfdd-06e0-4cd2-9407-e3ad60659aa3"
-					(reference "C_VDD_DOOR1")
+					(reference "C14")
 					(unit 1)
 				)
@@
 		(on_board yes)
 		(dnp no)
-		(property "Reference" "#PWR040"
+		(property "Reference" "#PWR041"
 			(at 193.04 73.66 0)
 			(effects
@@
 			(project "PROJECTE_EINES"
 				(path "/347831db-5db9-4aff-ad32-e56fd770e219/0182dfdd-06e0-4cd2-9407-e3ad60659aa3"
-					(reference "#PWR040")
+					(reference "#PWR041")
 					(unit 1)
 				)
@@
 		(on_board yes)
 		(dnp no)
-		(property "Reference" "C_WIN_1"
+		(property "Reference" "C8"
 			(at 48.006 44.196 90)
 			(effects
@@
 			(project "PROJECTE_EINES"
 				(path "/347831db-5db9-4aff-ad32-e56fd770e219/0182dfdd-06e0-4cd2-9407-e3ad60659aa3"
-					(reference "C_WIN_1")
+					(reference "C8")
 					(unit 1)
 				)
@@
 		(on_board yes)
 		(dnp no)
-		(property "Reference" "R_WIN_DIAGA1"
+		(property "Reference" "R10"
 			(at 95.758 66.802 90)
 			(effects
@@
 			(project "PROJECTE_EINES"
 				(path "/347831db-5db9-4aff-ad32-e56fd770e219/0182dfdd-06e0-4cd2-9407-e3ad60659aa3"
-					(reference "R_WIN_DIAGA1")
+					(reference "R10")
 					(unit 1)
 				)
@@
 		(on_board yes)
 		(dnp no)
-		(property "Reference" "C_VDD_DOOR2"
+		(property "Reference" "C15"
 			(at 163.068 58.42 90)
 			(effects
@@
 			)
 		)
-		(property "Footprint" "Capacitor_SMD:C_0805_2012Metric"
+		(property "Footprint" "Capacitor_SMD:C_1206_3216Metric"
 			(at 158.75 56.1848 0)
 			(effects
@@
 			(project "PROJECTE_EINES"
 				(path "/347831db-5db9-4aff-ad32-e56fd770e219/0182dfdd-06e0-4cd2-9407-e3ad60659aa3"
-					(reference "C_VDD_DOOR2")
+					(reference "C15")
 					(unit 1)
 				)
@@
 		(on_board yes)
 		(dnp no)
-		(property "Reference" "R_DIAGB_DOOR1"
+		(property "Reference" "R11"
 			(at 185.674 86.868 90)
 			(effects
@@
 			(project "PROJECTE_EINES"
 				(path "/347831db-5db9-4aff-ad32-e56fd770e219/0182dfdd-06e0-4cd2-9407-e3ad60659aa3"
-					(reference "R_DIAGB_DOOR1")
+					(reference "R11")
 					(unit 1)
 				)
@@
 		(on_board yes)
 		(dnp no)
-		(property "Reference" "C_WIN_2"
+		(property "Reference" "C9"
 			(at 47.498 54.61 90)
 			(effects
@@
 			)
 		)
-		(property "Footprint" "Capacitor_SMD:C_0805_2012Metric"
+		(property "Footprint" "Capacitor_SMD:C_1206_3216Metric"
 			(at 45.72 52.3748 0)
 			(effects
@@
 			(project "PROJECTE_EINES"
 				(path "/347831db-5db9-4aff-ad32-e56fd770e219/0182dfdd-06e0-4cd2-9407-e3ad60659aa3"
-					(reference "C_WIN_2")
+					(reference "C9")
 					(unit 1)
 				)
@@
 		(on_board yes)
 		(dnp no)
-		(property "Reference" "C_CP_DOOR1"
+		(property "Reference" "C18"
 			(at 185.42 60.96 90)
 			(effects
@@
 			(project "PROJECTE_EINES"
 				(path "/347831db-5db9-4aff-ad32-e56fd770e219/0182dfdd-06e0-4cd2-9407-e3ad60659aa3"
-					(reference "C_CP_DOOR1")
+					(reference "C18")
 					(unit 1)
 				)
@@
 		(dnp no)
 		(fields_autoplaced yes)
-		(property "Reference" "R_WIN_CS1"
+		(property "Reference" "R8"
 			(at 54.61 99.0599 0)
 			(effects
@@
 			(project "PROJECTE_EINES"
 				(path "/347831db-5db9-4aff-ad32-e56fd770e219/0182dfdd-06e0-4cd2-9407-e3ad60659aa3"
-					(reference "R_WIN_CS1")
-					(unit 1)
-				)
+					(reference "R8")
+					(unit 1)
+				)
