File: KiCad/PROJECTE_EINES.kicad_pcb (KiCad board)
At the start: 2 copper layers, 120.1 x 80.6 mm, 76 parts, among them J1 DE9_Pins_MountingHoles, J2 DE9_Pins_MountingHoles, J3 Conn_01x08_Pin, SW1 SW_DPDT_x2, SW2 SW_DPDT_x2, SW3 SW_DPDT_x2, U1 PIC24HJ128GP504-I_PT, U2 SN65HVD230, U3 VNH5019A-E, U4 LM2596S-5, U5 VNH5019A-E, U6 LM1117DT-3.3, Y1 8MHz

Commit message: Versio final KiCad, BOM i Diagrama de Blocs
Parts:
- removed R_CS_DOOR1: 1k, Resistor_SMD:R_0805_2012Metric
- added C2: 100n, Capacitor_SMD:C_0805_2012Metric, F.Cu at (153.8, 84.8)
- moved REF** 3.53 mm to (85.0, 100.4)
- moved REF** 1.08 mm to (197.8, 27.0)
- moved TP_5V1 0.90 mm to (127.0, 28.1)
- moved REF** 0.83 mm to (197.8, 100.4)
- moved TP_3V3 0.76 mm to (155.7, 28.1)
- moved REF** 0.54 mm to (84.8, 26.9)
- moved TP_PGEC1 0.50 mm to (147.6, 28.1)
- moved TP_PGED1 0.40 mm to (151.6, 27.8)
Connections:
- J3 pad 6: WIN_LIMIT -> +3.3V
- SW3 pad 2: unconnected-(SW3A-B-Pad2) -> GND
- U5 pad 6: GNDPWR -> +3.3V
- U5 pad 8: Net-(U5-CS) -> unconnected-(U5-CS-Pad8)
Routing:
- net +3.3V: track 267.4 -> 279.0 mm, vias 9 -> 10
- net GND: track 78.2 -> 85.0 mm
- net WIN_LIMIT: track 21.6 -> 27.8 mm
- net GNDPWR: track 146.9 -> 141.3 mm, vias 35 -> 32
- net Net-(U5-CS): track 4.38 -> 0.00 mm
- net +5V: track 46.9 -> 46.0 mm

Commit message: Afegida foodprint a R4 i actualitzada a la PCB
Parts:
- added R4: 10k, Resistor_SMD:R_0805_2012Metric, F.Cu at (145.8, 91.0)
Routing:
- net WIN_LIMIT: track 27.8 -> 34.0 mm
Changed lines of the file:
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@@
 		)
 	)
+	(footprint "Resistor_SMD:R_0805_2012Metric"
+		(layer "F.Cu")
+		(at 145.8 91)
+		(descr "Resistor SMD 0805 (2012 Metric), square (rectangular) end terminal, IPC-7351 nominal, (Body size source: IPC-SM-782 page 72, https://www.pcb-3d.com/wordpress/wp-content/uploads/ipc-sm-782a_amendment_1_and_2.pdf), generated with kicad-footprint-generator")
+		(tags "resistor")
+		(property "Reference" "R4"
+			(at 0 -1.65 0)
+			(layer "F.SilkS")
+			(effects
+				(font
+					(size 1 1)
+					(thickness 0.15)
+				)
+			)
+		)
+		(property "Value" "10k"
+			(at 0 1.65 0)
+			(layer "F.Fab")
+			(effects
+				(font
+					(size 1 1)
+					(thickness 0.15)
+				)
+			)
+		)
+		(property "Datasheet" "~"
+			(at 0 0 0)
+			(layer "F.Fab")
+			(hide yes)
+			(effects
+				(font
+					(size 1.27 1.27)
+					(thickness 0.15)
+				)
+			)
+		)
+		(property "Description" "Resistor"
+			(at 0 0 0)
+			(layer "F.Fab")
+			(hide yes)
+			(effects
+				(font
+					(size 1.27 1.27)
+					(thickness 0.15)
+				)
+			)
+		)
+		(property ki_fp_filters "R_*")
+		(sheetname "/SENSORS/")
+		(sheetfile "SENSOR_CORRENT.kicad_sch")
+		(attr smd)
+		(fp_line
+			(start -0.227064 -0.735)
+			(end 0.227064 -0.735)
+			(stroke
+				(width 0.12)
+				(type solid)
+			)
+			(layer "F.SilkS")
+		)
+		(fp_line
+			(start -0.227064 0.735)
+			(end 0.227064 0.735)
+			(stroke
+				(width 0.12)
+				(type solid)
+			)
+			(layer "F.SilkS")
+		)
+		(fp_rect
+			(start -1.68 -0.95)
+			(end 1.68 0.95)
+			(stroke
+				(width 0.05)
+				(type solid)
+			)
+			(fill no)
+			(layer "F.CrtYd")
+		)
+		(fp_rect
+			(start -1 -0.625)
+			(end 1 0.625)
+			(stroke
+				(width 0.1)
+				(type solid)
+			)
+			(fill no)
+			(layer "F.Fab")
+		)
+		(fp_text user "${REFERENCE}"
+			(at 0 0 0)
+			(layer "F.Fab")
+			(effects
+				(font
+					(size 0.5 0.5)
+					(thickness 0.08)
+				)
+			)
+		)
+		(pad "1" smd roundrect
+			(at -0.9125 0)
+			(size 1.025 1.4)
+			(layers "F.Cu" "F.Mask" "F.Paste")
+			(roundrect_rratio 0.243902)
+			(net 2 "+3.3V")
+			(pintype "passive")
+		)
+		(pad "2" smd roundrect
+			(at 0.9125 0)
+			(size 1.025 1.4)
+			(layers "F.Cu" "F.Mask" "F.Paste")
+			(roundrect_rratio 0.243902)
+			(net 38 "WIN_LIMIT")
+			(pintype "passive")
+		)
+		(embedded_fonts no)
+		(model "${KICAD9_3DMODEL_DIR}/Resistor_SMD.3dshapes/R_0805_2012Metric.step"
+			(offset
+				(xyz 0 0 0)
+			)
+			(scale
+				(xyz 1 1 1)
+			)
+			(rotate
+				(xyz 0 0 0)
+			)
+		)
+	)
 	(footprint "Package_SO:ST_MultiPowerSO-30"
 		(layer "F.Cu")
@@
 	)
 	(segment
+		(start 146.7125 91)
+		(end 152.8725 91)
+		(width 0.2)
+		(layer "F.Cu")
+		(net 38)
+	)
+	(segment
 		(start 152.9 91.0075)
 		(end 152.89 91.0175)
 		(width 0.2)
+		(layer "F.Cu")
+		(net 38)
+	)
+	(segment
+		(start 152.8725 91)
+		(end 152.89 91.0175)
+		(width 0.2)

Commit message: Versio final
Parts:
- CIN1, COUT1, C_VDD_DOOR2, C_WIN_2: footprint Capacitor_SMD:C_1206_3216Metric -> Capacitor_SMD:C_0805_2012Metric
- C_OSC1, C_OSC2: footprint Capacitor_SMD:C_0603_1608Metric -> Capacitor_SMD:C_0805_2012Metric

Commit message: Versió Final projecte
Parts:
- removed TP_3V3: TestPoint, TestPoint:TestPoint_Pad_D1.5mm
- added TP_3V1: TestPoint, TestPoint:TestPoint_Pad_D1.5mm, F.Cu at (164.0, 27.1)
- C1: renamed from C_OSC1; footprint Capacitor_SMD:C_0805_2012Metric -> Capacitor_SMD:C_0603_1608Metric
- C15: renamed from C_VDD_DOOR2; footprint Capacitor_SMD:C_0805_2012Metric -> Capacitor_SMD:C_1206_3216Metric
- C17: renamed from CIN1; footprint Capacitor_SMD:C_0805_2012Metric -> Capacitor_SMD:C_1206_3216Metric
- C19: renamed from COUT1; footprint Capacitor_SMD:C_0805_2012Metric -> Capacitor_SMD:C_1206_3216Metric
- C2: renamed from C_OSC2; footprint Capacitor_SMD:C_0805_2012Metric -> Capacitor_SMD:C_0603_1608Metric
- C9: renamed from C_WIN_2; footprint Capacitor_SMD:C_0805_2012Metric -> Capacitor_SMD:C_1206_3216Metric
- SW_UP1: value SW_MCLR -> SW
- moved TP_GND1 72.1 mm to (182.9, 27.1)
- moved TP_WDIAG1 24.3 mm to (121.8, 100.2)
- moved TP_MCLR1 19.2 mm to (156.8, 27.1)
- moved R13 15.5 mm to (159.9, 84.5), turned to 90 degrees
- moved TP_PGEC1 7.33 mm to (140.3, 27.1)
- moved TP_PGED1 3.27 mm to (148.4, 27.1)
- moved C15 2.22 mm to (107.2, 76.5)
- moved D2 2.16 mm to (92.0, 47.6)
- moved C8 1.29 mm to (120.0, 76.5)
- renumbered C_WIN_CP1 to C10, C_INBUCK1 to C11, C_INBUCK2 to C12, C_OUTBUCK1 to C13, C_VDD_DOOR1 to C14, C_OUTBUCK2 to C16, C_CP_DOOR1 to C18, COUT2 to C20, C2 to C21, C3 to C22, C_VDD2 to C3, C_AVDD1 to C4, C_BULK1 to C5, C_VCAP1 to C6, C1 to C7, C_WIN_1 to C8, D_PROT1 to D1, D_TVS1 to D2, D_OUTBUCK1 to D3, F_PROT1 to F1, R_WIN_DIAGA1 to R10, R_DIAGB_DOOR1 to R11, R_DIAGA_DOOR1 to R12, R4 to R13, R_MCLR1 to R4, R_BTNUP1 to R5, R_BTNDOWN1 to R6, R_Lock/Unlock1 to R7, R_WIN_CS1 to R8, R_WIN_DIAGB1 to R9
Routing:
- net WIN_DIAGA: track 42.7 -> 71.2 mm
- net +3.3V: track 279.0 -> 269.8 mm
- net WIN_LIMIT: track 34.0 -> 28.9 mm
- net PGEC1: track 36.0 -> 40.4 mm
- net MCLR: track 50.3 -> 54.1 mm, vias 0 -> 1
- net GND: track 85.0 -> 81.3 mm, vias 31 -> 30
- net VBAT_PROT: track 15.6 -> 13.5 mm
- net PGED1: track 34.8 -> 36.7 mm
- net GNDPWR: track 141.3 -> 141.8 mm, vias 32 -> 34
- added copper zone on F.Cu, net GND
Other:
- board text added: "Adrià Pelegrí i Gurpinder Singh"
- board text added: "MODUL DE CONTROL DE PORTA I FINESTRA"
- board text added: "PROJECTE EINES"
